File: Microphone Array CAD/Electrical/4-Channel Array/4-Channel Array/4-Channel Array.kicad_sch (KiCad schematic)
At the start: 20 parts, among them J1 Conn_01x05_Pin, U1 74LCX125MTCX

Commit message: Updated Array PCB
Parts:
- J1: footprint (none) -> Connector_JST:JST_XH_B5B-XH-A_1x05_P2.50mm_Vertical
Changed lines of the file:
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@@
 			)
 		)
-		(property "Footprint" ""
+		(property "Footprint" "Connector_JST:JST_XH_B5B-XH-A_1x05_P2.50mm_Vertical"
 			(at 138.43 144.78 0)
 			(effects
