File: Microphone Array CAD/Electrical/4-Channel Array/4-Channel Array/4-Channel Array.kicad_pcb (KiCad board)
At the start: 2 copper layers, 35 x 35 mm, 20 parts, among them J1 Conn_01x05_Pin, U1 74LCX125MTCX

Commit message: Continued development for Video
Parts:
- moved R8 63.7 mm to (181.0, 71.3), turned to 90 degrees
- moved R7 57.5 mm to (178.5, 61.3), turned to -90 degrees
Routing:
- net Net-(J1-Pin_5): track 0.00 -> 30.7 mm
- net Net-(U1-O0): track 0.00 -> 21.3 mm, vias 0 -> 2
- net Net-(J1-Pin_2): track 95.0 -> 108.5 mm, vias 1 -> 2
- net Net-(J1-Pin_3): track 13.7 -> 22.6 mm
- net Net-(MK3-DATA): track 0.00 -> 8.59 mm
- net Net-(U1-O3): track 0.00 -> 7.85 mm
- net Net-(J1-Pin_1): track 113.5 -> 119.8 mm, vias 1 -> 2
- net Net-(MK4-DATA): track 0.00 -> 5.71 mm
- net Net-(MK4-CLK): track 0.00 -> 4.06 mm
