File: Microphone Array CAD/Electrical/4-Channel Array/4-Channel Array V2/4-Channel Array V2/4-Channel Array V2.kicad_pcb (KiCad board)
At the start: 2 copper layers, 35 x 35 mm, 20 parts, among them J1 Conn_01x05_Pin, U1 74LCX125MTCX

Commit message: Continued Array Development
Parts:
- moved C3 15.5 mm to (168.5, 56.5), turned to 0 degrees
- moved R1 14.0 mm to (153.0, 70.8)
- moved C1 12.9 mm to (168.7, 68.0)
- moved J1 12.5 mm to (170.0, 52.5)
- moved R8 6.03 mm to (178.2, 66.0), turned to 180 degrees
- moved R3 4.56 mm to (179.2, 60.0), turned to 0 degrees
- moved R6 4.55 mm to (151.7, 66.0), turned to 0 degrees
- moved C2 4.25 mm to (154.0, 53.0), turned to 90 degrees
- moved R5 4.15 mm to (151.7, 64.0), turned to 0 degrees
- moved C5 2.83 mm to (177.5, 78.0), turned to -90 degrees
- moved R7 2.69 mm to (178.2, 64.0), turned to 180 degrees
- moved C4 2.69 mm to (152.5, 80.0), turned to -90 degrees
- moved R2 1.28 mm to (151.0, 74.0)
- moved C6 0.50 mm to (177.0, 52.0)
- moved U1 0.16 mm to (164.8, 72.5)
Routing:
- net Net-(MK1-CLK): track 4.30 -> 19.8 mm, vias 0 -> 2
- net Net-(J1-Pin_3): track 22.6 -> 37.3 mm, vias 4 -> 0
- net Net-(J1-Pin_2): track 131.4 -> 119.0 mm, vias 6 -> 4
- net Net-(U1-O0): track 20.3 -> 9.06 mm, vias 2 -> 0
- net Net-(U1-O2): track 29.2 -> 20.5 mm
- net Net-(MK4-DATA): track 5.71 -> 12.6 mm
- net Net-(J1-Pin_1): track 139.7 -> 146.5 mm, vias 6 -> 4
- net Net-(MK3-CLK): track 2.88 -> 8.17 mm
- net Net-(MK1-DATA): track 8.30 -> 12.5 mm
- net Net-(MK2-DATA): track 8.07 -> 11.8 mm
- net Net-(MK3-DATA): track 8.59 -> 11.9 mm
- net Net-(J1-Pin_4): track 21.3 -> 24.5 mm
- net Net-(U1-O1): track 11.6 -> 10.3 mm
- net Net-(J1-Pin_5): track 30.7 -> 31.6 mm, vias 0 -> 1

Commit message: Continued Array Development
Routing:
- net Net-(U1-O2): track 20.5 -> 19.6 mm
Other:
- outline, holes or cut-outs redrawn
Changed lines of the file:
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@@
 		(tags "resistor")
 		(property "Reference" "R7"
-			(at 0 1.5 360)
+			(at 0 1.5 0)
 			(layer "F.SilkS")
 			(effects
@@
 		)
 		(property "Value" "100 ohms"
-			(at 0 1.43 360)
+			(at 0 1.43 0)
 			(layer "F.Fab")
 			(hide yes)
@@
 		)
 		(fp_text user "${REFERENCE}"
-			(at 0 0 360)
+			(at 0 0 0)
 			(layer "F.Fab")
 			(effects
@@
 		(tags "resistor")
 		(property "Reference" "R5"
-			(at 0 -1.43 360)
+			(at 0 -1.43 0)
 			(layer "F.SilkS")
 			(effects
@@
 		)
 		(property "Value" "100 ohms"
-			(at 0 1.43 360)
+			(at 0 1.43 0)
 			(layer "F.Fab")
 			(hide yes)
@@
 		)
 		(fp_text user "${REFERENCE}"
-			(at 0 0 360)
+			(at 0 0 0)
 			(layer "F.Fab")
 			(effects
@@
 		(tags "resistor")
 		(property "Reference" "R3"
-			(at 0 -1.43 360)
+			(at 0 -1.43 0)
 			(layer "F.SilkS")
 			(effects
@@
 		)
 		(property "Value" "33 ohms"
-			(at -6.675 15.5 360)
+			(at -6.675 15.5 0)
 			(layer "F.Fab")
 			(hide yes)
@@
 		)
 		(fp_text user "${REFERENCE}"
-			(at 0 0 360)
+			(at 0 0 0)
 			(layer "F.Fab")
 			(effects
@@
 		(tags "resistor")
 		(property "Reference" "R8"
-			(at 0 -1.43 360)
+			(at 0 -1.43 0)
 			(layer "F.SilkS")
 			(effects
@@
 		)
 		(property "Value" "100 ohms"
-			(at 0 1.43 360)
+			(at 0 1.43 0)
 			(layer "F.Fab")
 			(hide yes)
@@
 		)
 		(fp_text user "${REFERENCE}"
-			(at 0 0 360)
+			(at 0 0 0)
 			(layer "F.Fab")
 			(effects
@@
 		(tags "resistor")
 		(property "Reference" "C3"
-			(at 0 -1.43 360)
+			(at 0 -1.43 0)
 			(layer "F.SilkS")
 			(effects
@@
 		)
 		(property "Value" "1uF"
-			(at 0 1.43 360)
+			(at 0 1.43 0)
 			(layer "F.Fab")
 			(hide yes)
@@
 		)
 		(fp_text user "${REFERENCE}"
-			(at 0 0 360)
+			(at 0 0 0)
 			(layer "F.Fab")
 			(effects
@@
 		(tags "resistor")
 		(property "Reference" "R6"
-			(at 0 1.5 360)
+			(at 0 1.5 0)
 			(layer "F.SilkS")
 			(effects
@@
 		)
 		(property "Value" "100 ohms"
-			(at 0 1.43 360)
+			(at 0 1.43 0)
 			(layer "F.Fab")
 			(hide yes)
@@
 		)
 		(fp_text user "${REFERENCE}"
-			(at 0 0 360)
+			(at 0 0 0)
 			(layer "F.Fab")
 			(effects
@@
 		(tags "resistor")
 		(property "Reference" "R2"
-			(at 0 -1.43 360)
+			(at 0 -1.43 0)
 			(layer "F.SilkS")
 			(effects
@@
 		)
 		(property "Value" "33 ohms"
-			(at 0 1.43 360)
+			(at 0 1.43 0)
 			(layer "F.Fab")
 			(hide yes)
@@
 		)
 		(fp_text user "${REFERENCE}"
-			(at 0 0 360)
+			(at 0 0 0)
 			(layer "F.Fab")
 			(effects
@@
 	)
 	(gr_line
+		(start 165 60)
+		(end 165 65)
+		(stroke
+			(width 0.1)
+			(type default)
+		)
+		(layer "Dwgs.User")
+	)
+	(gr_line
 		(start 180 80)
 		(end 150 80)
@@
 		(layer "Dwgs.User")
 	)
+	(gr_circle
+		(center 165 78.5)
+		(end 166.3 78.5)
+		(stroke
+			(width 0.05)
+			(type default)
+		)
+		(fill none)
+		(layer "Edge.Cuts")
+	)
 	(gr_line
 		(start 182.5 82.5)
@@
 		(layer "Edge.Cuts")
 	)
+	(gr_circle
+		(center 174.5 60)
+		(end 175.8 60)
+		(stroke
+			(width 0.05)
+			(type default)
+		)
+		(fill none)
+		(layer "Edge.Cuts")
+	)
 	(gr_line
 		(start 150 47.5)
@@
 	)
 	(gr_line
+		(start 155.5 60)
+		(end 174.5 60)
+		(stroke
+			(width 0.05)
+			(type default)
+		)
+		(layer "Edge.Cuts")
+	)
+	(gr_line
 		(start 182.5 47.5)
 		(end 182.5 82.5)
@@
 		(layer "Edge.Cuts")
 	)
+	(gr_circle
+		(center 155.5 60)
+		(end 156.8 60)
+		(stroke
+			(width 0.05)
+			(type default)
+		)
+		(fill none)
+		(layer "Edge.Cuts")
+	)
 	(gr_line
 		(start 147.5 47.5)
@@
 	)
 	(segment
-		(start 172.0442 72.4558)
-		(end 167.6896 72.4558)
+		(start 178 60)
+		(end 173.5 64.5)
 		(width 0.2)
 		(layer "F.Cu")
@@
 	(segment
 		(start 178.35 60)
-		(end 176.5 60)
+		(end 178 60)
 		(width 0.2)
 		(layer "F.Cu")
@@
 	)
 	(segment
-		(start 173.5 63)
+		(start 173.5 64.5)
 		(end 173.5 71)
 		(width 0.2)
@@
 	)
 	(segment
-		(start 176.5 60)
-		(end 173.5 63)
+		(start 173.5 71)
+		(end 172.0442 72.4558)
 		(width 0.2)
 		(layer "F.Cu")
@@
 	)
 	(segment
-		(start 173.5 71)
-		(end 172.0442 72.4558)
+		(start 172.0442 72.4558)
+		(end 167.6896 72.4558)
 		(width 0.2)
 		(layer "F.Cu")
